Commit message: Add ros2 control to robot (problem with wheels)

File: description/ros2_control.xacro (robot description, xacro)
@@ -1,4 +1,33 @@
 <?xml version="1.0"?>
 <robot xmlns:xacro="http://www.ros.org/wiki/xacro">
+    <ros2_control name="RealRobot" type="system">
+        <hardware>
+            <plugin>hoverboard_driver/hoverboard_driver</plugin>
+            <param name="wheel_radius">0.1</param>
+            <param name="max_velocity">1.0</param>
+            <param name="device">/dev/serial/by-id/usb-1a86_USB_Serial-if00-port0</param>
+        </hardware>
+        <joint name="left_wheel_joint">
+            <command_interface name="velocity">
+                <!--
+                <param name="min">-10</param>
+                <param name="max">10</param>
+                -->
+            </command_interface>
+            <state_interface name="position"/>
+            <state_interface name="velocity"/>
+        </joint>
+        <joint name="right_wheel_joint">
+            <command_interface name="velocity">
+                <!--
+                <param name="min">-10</param>
+                <param name="max">10</param>
+                -->
+            </command_interface>
+            <state_interface name="position"/>
+            <state_interface name="velocity"/>
+        </joint>
+    </ros2_control>
+    <!--
     <ros2_control name="GazeboSystem" type="system">
         <hardware>
@@ -27,3 +56,4 @@
         </plugin>
     </gazebo>
+    -->
 </robot>
